Commit message: dwa and pid now work together, needs tuning

File: robot-description/urdf/rikkert.urdf (robot description, URDF)
Before this commit: robot rikkert, 7 links, 6 joints
Links:
- link rear_caster: geometry collision sphere radius=0.08; visual sphere radius=0.08
Joints:
- joint caster_joint: axis 0 1 0 -> 1 1 0; type continuous -> revolute
