Commit message: Added urdf of rikkert

File: dif_robot.urdf (robot description, URDF)
Before this commit: robot dif_robot, 5 links, 4 joints
Links:
- link caster_wheel: geometry collision sphere radius=0.05; visual sphere radius=0.1
Joints:
- joint base_caster_wheel_joint: type continuous -> fixed

Commit message: Caster wheel changed

File: dif_robot.urdf (robot description, URDF)
Before this commit: robot dif_robot, 5 links, 4 joints
Joints:
- joint base_caster_wheel_joint: axis 0 1 0 -> 1 1 0; type fixed -> revolute

File: robot-description/urdf/rikkert.urdf (robot description, URDF)
Before this commit: robot rikkert, 7 links, 6 joints
Links:
- removed link rear_caster
- added link caster_body, mass 0.4; collision cylinder length=0.08 radius=0.05; visual cylinder length=0.08 radius=0.05
- added link caster_wheel, mass 0.25; collision cylinder length=0.04 radius=0.06; visual cylinder length=0.04 radius=0.06
- link base_link: mass 0.4 -> 2
Joints:
- removed joint caster_joint
- added joint caster_rolling_joint: type revolute, parent caster_body, child caster_wheel, origin xyz=0 0 -0.06 rpy=0 0 0, axis 0 1 0, limit lower=-100000000 upper=100000000 effort=100 velocity=10
- added joint caster_swivel_joint: type continuous, parent base_link, child caster_body, origin xyz=-0.285 0 -0.03 rpy=0 0 0, axis 0 0 1

Commit message: Debugging physics

File: dif_robot.urdf (robot description, URDF)
Before this commit: robot dif_robot, 5 links, 4 joints
Links:
- added link caster_body, mass 0.4; collision cylinder length=0.08 radius=0.05; visual cylinder length=0.08 radius=0.05
- link caster_wheel: mass 2 -> 0.25; geometry collision cylinder length=0.04 radius=0.06; visual cylinder length=0.04 radius=0.06
Joints:
- removed joint base_caster_wheel_joint
- added joint caster_rolling_joint: type revolute, parent caster_body, child caster_wheel, origin xyz=0 0 -0.06 rpy=0 0 0, axis 0 1 0, limit lower=-100000000 upper=100000000 effort=50 velocity=10
- added joint caster_swivel_joint: type continuous, parent base_link, child caster_body, origin xyz=0.2 0 -0.03 rpy=0 0 0, axis 0 0 1
- joint base_left_wheel_joint: limit lower=-100000000 upper=100000000 effort=500 velocity=500 -> lower=-100000000 upper=100000000 effort=50 velocity=500
- joint base_right_wheel_joint: limit lower=-100000000 upper=100000000 effort=500 velocity=500 -> lower=-100000000 upper=100000000 effort=50 velocity=500

File: robot-description/urdf/rikkert.urdf (robot description, URDF)
Before this commit: robot rikkert, 8 links, 7 joints
Links:
- link caster_body: mass 0.4 -> 0.8
- link left_wheel: mass 0.1105 -> 5
- link right_wheel: mass 0.1105 -> 5
Joints:
- joint caster_rolling_joint: limit lower=-100000000 upper=100000000 effort=100 velocity=10 -> lower=-100000000 upper=100000000 effort=10000 velocity=10
- joint caster_swivel_joint: limit (none) -> lower=-100000000 upper=100000000 effort=1000 velocity=10

Commit message: config en urdf aanpassingen voor smoothness

File: dif_robot.urdf (robot description, URDF)
Before this commit: robot dif_robot, 5 links, 4 joints
Joints:
- removed joint base_left_wheel_joint
- removed joint base_right_wheel_joint
- added joint left_wheel_joint: type continuous, parent base_link, child left_wheel, origin xyz=-0.15 0.225 0 rpy=0 0 0, axis 0 1 0, limit lower=-100000000 upper=100000000 effort=500 velocity=500
- added joint right_wheel_joint: type continuous, parent base_link, child right_wheel, origin xyz=-0.15 -0.225 0 rpy=0 0 0, axis 0 1 0, limit lower=-100000000 upper=100000000 effort=500 velocity=500
- joint base_caster_wheel_joint: axis 0 1 0 -> 1 1 0; type fixed -> revolute

File: robot-description/urdf/rikkert.urdf (robot description, URDF)
Before this commit: robot rikkert, 7 links, 6 joints
Links:
- removed link base_footprint
- removed link hokuyo
- removed link rear_caster
- removed link rs_bpearl
- added link caster_wheel, mass 2; collision sphere radius=0.05; visual sphere radius=0.1
- added link lidar_link, mass 0.1; visual cylinder length=0.05 radius=0.1
- link base_link: mass 0.4 -> 10.0; geometry collision box size=0.6 0.4 0.2; visual box size=0.6 0.4 0.2
- link left_wheel: mass 0.1105 -> 5; geometry collision cylinder length=0.05 radius=0.1; visual cylinder length=0.05 radius=0.1
- link right_wheel: mass 0.1105 -> 5; geometry collision cylinder length=0.05 radius=0.1; visual cylinder length=0.05 radius=0.1
Joints:
- removed joint bpearl_joint
- removed joint caster_joint
- removed joint footprint_base
- removed joint hokuyo_joint
- added joint base_caster_wheel_joint: type revolute, parent base_link, child caster_wheel, origin xyz=-0.2 0.0 -0.05 rpy=0.0 0.0 0.0, axis 1 1 0, limit lower=-100000000 upper=100000000 effort=100 velocity=100
- added joint base_lidar_joint: type fixed, parent base_link, child lidar_link, origin xyz=0 0 0.225
- joint left_wheel_joint: limit lower=-100000000 upper=100000000 effort=1000 velocity=100000000 -> lower=-100000000 upper=100000000 effort=500 velocity=500; origin xyz=0.28 0.285 0.05 rpy=0 0 0 -> xyz=0.15 0.225 0 rpy=0 0 0
- joint right_wheel_joint: limit lower=-100000000 upper=100000000 effort=1000 velocity=100000000 -> lower=-100000000 upper=100000000 effort=500 velocity=500; origin xyz=0.28 -0.285 0.05 rpy=0 0 0 -> xyz=0.15 -0.225 0 rpy=0 0 0
